File: board/uf2-batch-flasher/level2.kicad_sch (KiCad schematic)
At the start: 2 parts, among them U102 FSUSB74

Commit message: Briefly document and add the OSHW logo.
Other:
- company: (none) -> nbp.name
- title: (none) -> UF2 Batch Flasher
Changed lines of the file:
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@@
 (kicad_sch (version 20230121) (generator eeschema)
   (paper "A4")
+  (title_block
+    (title "UF2 Batch Flasher")
+    (date "2023-10-20")
+    (rev "0.1")
+    (company "nbp.name")
+    (comment 2 "are dispatched to the leaves of the tree of USB devices.")
+    (comment 3 "This is the third level, where select flags and data lines")
+    (comment 4 "UF2 Batch Flasher is a USB hub for flashing USB devices")
+  )
   (junction (at 173.99 77.47) (diameter 0) (color 0 0 0 0)
   )

Commit message: Fix Select pins mapping.
Both the selector and demultiplexer are used to enable/disable the power
and data pins. If the mapping of pins is not identical between the 2
then we would enable the power pins of one USB port and the data pins of
another.

This patch changes that such that components which are closer to the
Pico are using the high-power bits while components which are further
down the tree are using the low bits. This way the enable pins are
correctly ordered as specified in the datasheets of both components.

Previously we were using the lowest bits, this would have been if
the enable pins were mapped accordingly. Which was not the case.

This change include changes in the schematics and in the board layout.
The component remain at their original placement.

This change also adds the OSHW logo as well as the fiducial in the
schematic such that they are not removed each time we re-import the
schematics in the board.
Connections:
- net SEL4 renamed SEL0
- net SEL5 renamed SEL1
Changed lines of the file:
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@@
     (effects (font (size 1.27 1.27)) (justify left))
   )
-  (hierarchical_label "SEL4" (shape input) (at 171.45 74.93 180) (fields_autoplaced)
+  (hierarchical_label "SEL0" (shape input) (at 171.45 74.93 180) (fields_autoplaced)
     (effects (font (size 1.27 1.27)) (justify right))
   )
-  (hierarchical_label "SEL5" (shape input) (at 171.45 77.47 180) (fields_autoplaced)
+  (hierarchical_label "SEL1" (shape input) (at 171.45 77.47 180) (fields_autoplaced)
     (effects (font (size 1.27 1.27)) (justify right))
   )
