File: board/uf2-batch-flasher/usb-port.kicad_sch (KiCad schematic)
At the start: 14 parts, among them J101 USB_A, U401 AP22804AW5-7

Commit message: Briefly document and add the OSHW logo.
Other:
- company: (none) -> nbp.name
- title: (none) -> UF2 Batch Flasher
Changed lines of the file:
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@@
 (kicad_sch (version 20230121) (generator eeschema)
   (paper "A4")
+  (title_block
+    (title "UF2 Batch Flasher")
+    (date "2023-10-20")
+    (rev "0.1")
+    (company "nbp.name")
+    (comment 2 "as well as some ESD protection on the data lines.")
+    (comment 3 "This page contains a single USB port, with the essential components needed to enable it,")
+    (comment 4 "UF2 Batch Flasher is a USB hub for flashing USB devices")
+  )
   (junction (at 187.96 115.57) (diameter 0) (color 0 0 0 0)
   )
